File: Scheda Hardware/Scheda Hardware.kicad_pcb (KiCad board)
At the start: 2 copper layers, 53.3 x 94 mm, 11 parts, among them SW1 SW_Push, SW2 SW_Push, U2 NodeMCU_1.0_(ESP-12E)

Commit message: update
Parts:
- added Brd1: SSD1306, SSD1306:128x64OLED, B.Cu at (138.4, 49.5)
- added H1: MountingHole, MountingHole:MountingHole_3.2mm_M3, F.Cu at (115.6, 39.4)
- added H2: MountingHole, MountingHole:MountingHole_3.2mm_M3, F.Cu at (115.6, 121.9)
- added H3: MountingHole, MountingHole:MountingHole_3.2mm_M3, F.Cu at (161.3, 39.4)
- added H4: MountingHole, MountingHole:MountingHole_3.2mm_M3, F.Cu at (161.3, 121.9)
- added R1: R, Resistor_THT:R_Axial_DIN0207_L6.3mm_D2.5mm_P10.16mm_Horizontal, F.Cu at (120.0, 101.6)
- added R2: R, Resistor_THT:R_Axial_DIN0207_L6.3mm_D2.5mm_P10.16mm_Horizontal, F.Cu at (156.2, 88.9)
- added RFID1: ~, RestRoomTime:RFID-RC522, B.Cu at (148.0, 125.7)
- added SW1: SW_Push, Button_Switch_SMD:SW_Push_1P1T_NO_6x6mm_H9.5mm, B.Cu at (118.7, 54.9)
- added SW2: SW_Push, Button_Switch_SMD:SW_Push_1P1T_NO_6x6mm_H9.5mm, B.Cu at (158.6, 55.0)
- added U2: NodeMCU_1.0_(ESP-12E), ESP8266:NodeMCU-LoLinV3, F.Cu at (138.4, 96.5)
Routing:
- net /SCL: track 147.4 -> 294.7 mm
- net /SDA: track 96.8 -> 193.7 mm
- net +3.3V: track 96.3 -> 192.6 mm
- net Net-(RFID1-RST): track 72.0 -> 144.0 mm
- net /P2: track 55.0 -> 110.0 mm
- net /MOSI: track 47.4 -> 94.9 mm
- net /P1: track 45.2 -> 90.4 mm
- net /MISO: track 42.0 -> 84.1 mm
Other:
- board size 53.3 x 94 mm -> 116.8 x 94 mm

Commit message: update
Parts:
- removed the Brd1 at (138.4, 49.5)
- removed the H1 at (115.6, 39.4)
- removed the H2 at (115.6, 121.9)
- removed the H3 at (161.3, 39.4)
- removed the H4 at (161.3, 121.9)
- removed the R1 at (120.0, 101.6)
- removed the R2 at (156.2, 88.9)
- removed the RFID1 at (148.0, 125.7)
- removed the SW1 at (118.7, 54.9)
- removed the SW2 at (158.6, 55.0)
- removed the U2 at (138.4, 96.5)
Routing:
- net /SCL: track 294.7 -> 147.4 mm
- net /SDA: track 193.7 -> 96.8 mm
- net +3.3V: track 192.6 -> 96.3 mm
- net Net-(RFID1-RST): track 144.0 -> 72.0 mm
- net /P2: track 110.0 -> 55.0 mm
- net /MOSI: track 94.9 -> 47.4 mm
- net /P1: track 90.4 -> 45.2 mm
- net /MISO: track 84.1 -> 42.0 mm
Other:
- board size 116.8 x 94 mm -> 53.3 x 94 mm
