File: Scheda Hardware/Scheda Hardware.kicad_sch (KiCad schematic)
At the start: 11 parts, among them SW1 SW_Push, SW2 SW_Push, U2 NodeMCU_1.0_(ESP-12E)

Commit message: update
Other:
- note added: "MISO"
- note added: "MOSI"
Changed lines of the file:
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@@
     (stroke (width 0) (type default))
+  )
+  (text "MOSI" (at 109.22 59.69 0)
+    (effects (font (size 1.27 1.27)) (justify left bottom))
+  )
+  (text "MISO" (at 109.22 57.15 0)
+    (effects (font (size 1.27 1.27)) (justify left bottom))
   )
   (label "SCL" (at 111.76 39.37 0) (fields_autoplaced)
